File: BeerBoard-stand.kicad_sch (KiCad schematic)
At the start: 12 parts, among them J1 Conn_02x04_Odd_Even

Commit message: Some updates, added images
Parts:
- added C1, C10: 3u3, Capacitor_SMD:C_0805_2012Metric_Pad1.18x1.45mm_HandSolder, symbol Device:C
- added C2, C3: 390p, Capacitor_SMD:C_0603_1608Metric_Pad1.08x0.95mm_HandSolder, symbol Device:C
- added C4, C5, C6, C9: 1u, Capacitor_SMD:C_0805_2012Metric_Pad1.18x1.45mm_HandSolder, symbol Device:C
- added C7, C8: 100n, Capacitor_SMD:C_0603_1608Metric_Pad1.08x0.95mm_HandSolder, symbol Device:C
- added D6: D_Zener, Diode_THT:D_DO-35_SOD27_P7.62mm_Horizontal, symbol Device:D_Zener
- added D7: LED, LED_SMD:LED_0805_2012Metric_Pad1.15x1.40mm_HandSolder, symbol Device:LED
- added H1, H2, H3: MountingHole, MountingHole:MountingHole_3.2mm_M3, symbol Mechanical:MountingHole
- added J2: Type-C_6P, Connector_USB:USB_C_Receptacle_GCT_USB4125-xx-x-0190_6P_TopMnt_Horizontal, symbol Connector:USB_C_Receptacle_PowerOnly_6P
- added J3: I2C, Connector_PinHeader_2.54mm:PinHeader_1x02_P2.54mm_Vertical, symbol Connector_Generic:Conn_01x02
- added J4: Conn_01x03, Connector_PinHeader_2.54mm:PinHeader_1x03_P2.54mm_Vertical, symbol Connector_Generic:Conn_01x03
- added JP1: SolderJumper_2_Open, Jumper:SolderJumper-2_P1.3mm_Open_RoundedPad1.0x1.5mm, symbol Jumper:SolderJumper_2_Open
- added JP2, JP3: SolderJumper_3_Bridged12, Jumper:SolderJumper-3_P1.3mm_Bridged2Bar12_RoundedPad1.0x1.5mm_NumberLabels, symbol Jumper:SolderJumper_3_Bridged12
- added Q1: DMP3098LSD, Package_SO:SOIC-8-1EP_3.9x4.9mm_P1.27mm_EP2.29x3mm, symbol Device:Q_Dual_PMOS_S1G1S2G2D2D2D1D1
- added R10, R20, R23: 1k, Resistor_SMD:R_0603_1608Metric, symbol Device:R
- added R11, R12, R19, R22: 2k4, Resistor_SMD:R_0603_1608Metric, symbol Device:R
- added R13, R14, R15, R16, R18, R21: 5k1, Resistor_SMD:R_0603_1608Metric, symbol Device:R
- added R17, R7: 10k, Resistor_SMD:R_0603_1608Metric, symbol Device:R
- added R24: 0, Resistor_SMD:R_0603_1608Metric, symbol Device:R
- added R8: 50K, Resistor_SMD:R_0603_1608Metric, symbol Device:R
- added R9: 1K, Resistor_SMD:R_0603_1608Metric, symbol Device:R
- added SW1, SW2: ~, USB:SK-14D01-G 6, symbol New_Library:SW_SP4T
- added TP1, TP2, TP3: TestPoint, TestPoint:TestPoint_Pad_1.0x1.0mm, symbol Connector:TestPoint
- added U1: CYPD3177-24LQ, Package_DFN_QFN:QFN-24-1EP_4x4mm_P0.5mm_EP2.75x2.75mm, symbol New_Library:CYPD3177
- R6: value 100k -> 50k
Connections:
- net GND: now also C1.2, C10.2, C2.2, C3.2, C6.2, C7.2, C8.2, C9.2, D7.1 (K), J2.A12 (GND), J2.B12 (GND), J4.1 (Pin_1), JP1.2 (B), R14.2, R15.2, R17.2, R18.2, R19.2, R20.2, R21.2, R22.2, R23.2, R24.2, U1.19 (GND), U1.22 (GND), U1.25 (GND)
- net VDD: now also R11.1, R12.1
- new net: D7.2 (A), R10.1
- new net: R10.2, TP2.1, U1.9 (FAULT)
- new net: JP3.1 (A), SW2.3, SW2.4
- new net: JP3.2 (C), R16.2, U1.2 (VBUS_MAX)
- new net: JP3.3 (B), R24.1
- new net: C4.2, C5.2, D6.2 (A), Q1.2 (G), Q1.4 (G), R7.2, R8.2, R9.1
- new net: R21.1, SW2.5
- new net: R15.1, U1.1 (VBUS_MIN)
- new net: R9.2, U1.3 (VBUS_FET_EN)
- new net: J3.1 (Pin_1), R12.2, U1.12 (HPI_SDA)
- new net: J3.2 (Pin_2), R11.2, U1.13 (HPI_SCL)
- new net: TP3.1, U1.10 (FLIP)
- new net: C3.1, J2.B5 (CC2), U1.14 (CC2)
- new net: C2.1, J2.A5 (CC1), U1.15 (CC1)
- new net: C9.1, U1.24 (VCCD)
- new net: TP1.1, U1.4 (SAFE_PWR_EN)
- new net: JP2.2 (C), R13.2, U1.5 (ISNK_COARSE)
- new net: R14.1, U1.6 (ISNK_FINE)
- new net: D6.1 (K), Q1.1 (S), Q1.3 (S), R8.1
- new net: J2.S1 (SHIELD), JP1.1 (A)
- new net: JP2.1 (A), SW1.3, SW1.4
- new net: JP2.3 (B), R20.1
- new net: R23.1, SW2.1
- new net: R22.1, SW2.2
- new net: R19.1, SW1.1
- new net: R18.1, SW1.2
- new net: R17.1, SW1.5
- new net +3V3: C6.1, C7.1, C8.1, R13.1, R16.1, U1.23 (VDDD)
- new net +VSW: C10.1, C5.1, J4.2 (Pin_2), J4.3 (Pin_3), Q1.5 (D), Q1.6 (G), U1.11 (VDC_OUT)
- new net VBUS: C1.1, C4.1, J2.A9 (VBUS), J2.B9 (VBUS), Q1.7 (D), Q1.8 (G), R7.1, U1.18 (VBUS_IN)
- no-connect marks 0 -> 4
Other:
- note added: "12V"
- note added: "15V"
- note added: "1A"
- note added: "20V"
- note added: "2A"
- note added: "3A"
- note added: "4A"
- note added: "5A"
- note added: "5V"
- note added: "9V"
- note added: "Header (BeerBoard-stand)"
- note added: "LEDs (BeerBoard-stand)"
- note added: "USB-C PD"
- note removed: "Header"
- note removed: "LEDs"
- moved on the sheet: D2, D3, D4, D5, J1, R1, R2, R3, R4, R5, R6
